Commit message: Add fire_B horizontal disk sweep project

File: src/robot/urdf/robot.urdf (robot description, URDF)
Before this commit: robot robot, 8 links, 7 joints
Joints:
- joint base_joint: limit lower=-3 upper=3 effort=200 velocity=5 -> lower=-3 upper=3 effort=200 velocity=25
- joint elbow_joint: limit lower=-3 upper=3 effort=200 velocity=5 -> lower=-3 upper=3 effort=200 velocity=25
- joint shoulder_joint: limit lower=-3 upper=3 effort=200 velocity=5 -> lower=-3 upper=3 effort=200 velocity=25
- joint wrist1_joint: limit lower=-3 upper=3 effort=200 velocity=5 -> lower=-3 upper=3 effort=200 velocity=25
- joint wrist2_joint: limit lower=-3 upper=3 effort=200 velocity=5 -> lower=-3 upper=3 effort=200 velocity=25
- joint wrist3_joint: limit lower=-3 upper=3 effort=200 velocity=5 -> lower=-3 upper=3 effort=200 velocity=25
